Commit message: Matched pinocchio pendulum with previous version (minus integration)

File: examples/urdf/pendulum.urdf (robot description, URDF)
Before this commit: robot omnipointer, 2 links, 1 joints
Joints:
- joint pendulum_joint_1: limit lower=-12. upper=12 effort=2.5 velocity=10.0 -> lower=-10000. upper=10000 effort=7 velocity=10000.0
