Commit message: Improved solution saving to file & added viser for visualization

File: examples/urdf/a1/a1.urdf (robot description, URDF)
Before this commit: robot a1_description, 18 links, 17 joints
Links:
- link FL_calf: geometry collision box size=0.2 0.016 0.016; visual mesh filename=./a1_description/meshes/calf.glb scale=1 1 1
- link FL_hip: geometry collision cylinder length=0.04 radius=0.046; visual mesh filename=./a1_description/meshes/hip.glb scale=1 1 1
- link FL_thigh: geometry collision box size=0.2 0.0245 0.034; visual mesh filename=./a1_description/meshes/thigh.glb scale=1 1 1
- link FR_calf: geometry collision box size=0.2 0.016 0.016; visual mesh filename=./a1_description/meshes/calf.glb scale=1 1 1
- link FR_hip: geometry collision cylinder length=0.04 radius=0.046; visual mesh filename=./a1_description/meshes/hip.glb scale=1 1 1
- link FR_thigh: geometry collision box size=0.2 0.0245 0.034; visual mesh filename=./a1_description/meshes/thigh_mirror.glb scale=1 1 1
- link RL_calf: geometry collision box size=0.2 0.016 0.016; visual mesh filename=./a1_description/meshes/calf.glb scale=1 1 1
- link RL_hip: geometry collision cylinder length=0.04 radius=0.046; visual mesh filename=./a1_description/meshes/hip.glb scale=1 1 1
- link RL_thigh: geometry collision box size=0.2 0.0245 0.034; visual mesh filename=./a1_description/meshes/thigh.glb scale=1 1 1
- link RR_calf: geometry collision box size=0.2 0.016 0.016; visual mesh filename=./a1_description/meshes/calf.glb scale=1 1 1
- link RR_hip: geometry collision cylinder length=0.04 radius=0.046; visual mesh filename=./a1_description/meshes/hip.glb scale=1 1 1
- link RR_thigh: geometry collision box size=0.2 0.0245 0.034; visual mesh filename=./a1_description/meshes/thigh_mirror.glb scale=1 1 1
- link trunk: geometry collision box size=0.267 0.194 0.114; visual mesh filename=./a1_description/meshes/trunk.glb scale=1 1 1

File: examples/urdf/panda/panda.urdf (robot description, URDF)
Before this commit: robot panda, 13 links, 12 joints
Links:
- link panda_hand: geometry collision mesh filename=./panda_description/meshes/collision/hand.stl; visual mesh filename=./panda_description/meshes/visual/hand.dae
- link panda_leftfinger: geometry collision mesh filename=./panda_description/meshes/collision/finger.stl; visual mesh filename=./panda_description/meshes/visual/finger.dae
- link panda_link0: geometry collision mesh filename=./panda_description/meshes/collision/link0.stl; visual mesh filename=./panda_description/meshes/visual/link0.dae
- link panda_link1: geometry collision mesh filename=./panda_description/meshes/collision/link1.stl; visual mesh filename=./panda_description/meshes/visual/link1.dae
- link panda_link2: geometry collision mesh filename=./panda_description/meshes/collision/link2.stl; visual mesh filename=./panda_description/meshes/visual/link2.dae
- link panda_link3: geometry collision mesh filename=./panda_description/meshes/collision/link3.stl; visual mesh filename=./panda_description/meshes/visual/link3.dae
- link panda_link4: geometry collision mesh filename=./panda_description/meshes/collision/link4.stl; visual mesh filename=./panda_description/meshes/visual/link4.dae
- link panda_link5: geometry collision mesh filename=./panda_description/meshes/collision/link5.stl; visual mesh filename=./panda_description/meshes/visual/link5.dae
- link panda_link6: geometry collision mesh filename=./panda_description/meshes/collision/link6.stl; visual mesh filename=./panda_description/meshes/visual/link6.dae
- link panda_link7: geometry collision mesh filename=./panda_description/meshes/collision/link7.stl; visual mesh filename=./panda_description/meshes/visual/link7.dae
- link panda_rightfinger: geometry collision mesh filename=./panda_description/meshes/collision/finger.stl; visual mesh filename=./panda_description/meshes/visual/finger.dae
