Commit message: Improved visualizer, added talos standing example (c++)

File: examples/urdf/talos/talos.urdf (robot description, URDF)
Before this commit: robot talos, 60 links, 59 joints
Links:
- added link left_mm
- added link left_mp
- added link left_pm
- added link left_pp
- added link right_mm
- added link right_mp
- added link right_pm
- added link right_pp
Joints:
- added joint left_mm_fix_joint: type fixed, parent leg_left_6_link, child left_mm, origin xyz=-0.1105 -0.067 -0.107 rpy=0 0 0
- added joint left_mp_fix_joint: type fixed, parent leg_left_6_link, child left_mp, origin xyz=-0.1105 0.067 -0.107 rpy=0 0 0
- added joint left_pm_fix_joint: type fixed, parent leg_left_6_link, child left_pm, origin xyz=0.1105 -0.067 -0.107 rpy=0 0 0
- added joint left_pp_fix_joint: type fixed, parent leg_left_6_link, child left_pp, origin xyz=0.1105 0.067 -0.107 rpy=0 0 0
- added joint right_mm_fix_joint: type fixed, parent leg_right_6_link, child right_mm, origin xyz=-0.1105 -0.067 -0.107 rpy=0 0 0
- added joint right_mp_fix_joint: type fixed, parent leg_right_6_link, child right_mp, origin xyz=-0.1105 0.067 -0.107 rpy=0 0 0
- added joint right_pm_fix_joint: type fixed, parent leg_right_6_link, child right_pm, origin xyz=0.1105 -0.067 -0.107 rpy=0 0 0
- added joint right_pp_fix_joint: type fixed, parent leg_right_6_link, child right_pp, origin xyz=0.1105 0.067 -0.107 rpy=0 0 0
