Commit message: Added initial MPC pendubot example

File: examples/urdf/double_pendulum/double_pendulum_2.urdf (robot description, URDF)
Before this commit: robot double_pendulum, 5 links, 4 joints
Joints:
- joint joint1: limit lower=-3.14 upper=3.14 effort=0.05 velocity=25 -> lower=-3.14 upper=3.14 effort=0.15 velocity=25
- joint joint2: limit lower=-3.14 upper=3.14 effort=0.05 velocity=35 -> lower=-3.14 upper=3.14 effort=0.15 velocity=35

Commit message: Exposed SSQP and ADMM params structs in the Python API, added SSQP line-search regularization-related parameters, improved pendubot example

File: examples/urdf/double_pendulum/double_pendulum_2.urdf (robot description, URDF)
Before this commit: robot double_pendulum, 5 links, 4 joints
Joints:
- joint joint1: limit lower=-3.14 upper=3.14 effort=0.15 velocity=25 -> lower=-10000 upper=10000 effort=0.15 velocity=25
- joint joint2: limit lower=-3.14 upper=3.14 effort=0.15 velocity=35 -> lower=-10000 upper=10000 effort=0.15 velocity=35

Commit message: Added vector weight option for various predefined costs

File: examples/urdf/double_pendulum/double_pendulum_2.urdf (robot description, URDF)
Before this commit: robot double_pendulum, 5 links, 4 joints
Links:
- added link tip; visual sphere radius=0.006
- link joint2_sphere: geometry visual sphere radius=0.006
Joints:
- added joint tip_link: type fixed, parent link2, child tip, origin xyz=0 0 -0.05
- joint joint1: limit lower=-10000 upper=10000 effort=0.15 velocity=25 -> lower=-10000 upper=10000 effort=0.1 velocity=25
