Commit message: Tuned real system MPC for double pendulum (both joints actuated)

File: examples/urdf/double_pendulum/double_pendulum.urdf (robot description, URDF)
Before this commit: robot 2dof_planar, 3 links, 2 joints
Links:
- added link joint1_sphere; visual sphere radius=0.01
- added link joint2_sphere; visual sphere radius=0.006
- added link tip; visual sphere radius=0.006
- link base_link: mass 0.10159 -> None; geometry visual box size=0.015 0.015 0.015
- link link1: mass 0.26703 -> 0.10548177618443695; geometry visual cylinder length=0.05 radius=0.005
- link link2: mass 0.33238 -> 0.07619744360415454; geometry visual cylinder length=0.05 radius=0.005
Joints:
- added joint joint1_link: type fixed, parent joint1_sphere, child link1
- added joint joint2_link: type fixed, parent joint2_sphere, child link2
- added joint tip_link: type fixed, parent link2, child tip, origin xyz=0 0 -0.05
- joint joint1: child link1 -> joint1_sphere; limit lower=0 upper=0 effort=0 velocity=0 -> lower=-10000 upper=10000 effort=0.1 velocity=25; origin xyz=0.0060872 0 0.035 rpy=0 0 0 -> xyz=0 0 0
- joint joint2: child link2 -> joint2_sphere; limit lower=0 upper=0 effort=0 velocity=0 -> lower=-10000 upper=10000 effort=0.1 velocity=35; origin xyz=0.023 0 0.1 rpy=0 0 0 -> xyz=0 0 -0.05

File: examples/urdf/double_pendulum/pendubot.urdf (robot description, URDF)
Before this commit: robot double_pendulum, 6 links, 5 joints
Joints:
- joint joint2: limit lower=-10000 upper=10000 effort=0.15 velocity=35 -> lower=-10000 upper=10000 effort=0.0 velocity=35

Commit message: Tuned real system MPC for pendubot (one joint actuated) with ID

File: examples/urdf/double_pendulum/double_pendulum.urdf (robot description, URDF)
Before this commit: robot double_pendulum, 6 links, 5 joints
Joints:
- joint joint1: limit lower=-10000 upper=10000 effort=0.1 velocity=25 -> lower=-10000 upper=10000 effort=0.15 velocity=25
- joint joint2: limit lower=-10000 upper=10000 effort=0.1 velocity=35 -> lower=-10000 upper=10000 effort=0.15 velocity=35
