Commit message: Updated Pendubot and Panda real MPC scripts

File: examples/assets/urdf/double_pendulum/pendubot.urdf (robot description, URDF)
Before this commit: robot double_pendulum, 6 links, 5 joints
Joints:
- joint joint1: limit lower=-10000 upper=10000 effort=0.15 velocity=25 -> lower=-10000 upper=10000 effort=0.1 velocity=25

File: examples/assets/urdf/double_pendulum/pendubot_cont.urdf (robot description, URDF)
Before this commit: robot double_pendulum, 6 links, 5 joints
Joints:
- joint joint1: limit effort=0.15 velocity=25 -> effort=0.1 velocity=25
