Commit message: Added new general model methods for torque regressor matrix & dynamic parameters

File: examples/assets/urdf/double_pendulum/pendubot.urdf (robot description, URDF)
Before this commit: robot double_pendulum, 6 links, 5 joints
Joints:
- joint joint1: limit lower=-10000 upper=10000 effort=0.1 velocity=25 -> lower=-10000 upper=10000 effort=0.15 velocity=25

Commit message: Fixed simulation script for pendubot adaptive model updating & added same option for real MPC script

File: examples/assets/urdf/double_pendulum/pendubot.urdf (robot description, URDF)
Before this commit: robot double_pendulum, 6 links, 5 joints
Joints:
- joint joint1: limit lower=-10000 upper=10000 effort=0.15 velocity=25 -> lower=-10000 upper=10000 effort=0.1 velocity=25
- joint joint2: limit lower=-10000 upper=10000 effort=0.0 velocity=35 -> lower=-10000 upper=10000 effort=0.0 velocity=25

Commit message: Fixed Fatrop solver benchmark dockerfile & updated Pendubot real MPC scripts

File: examples/assets/urdf/double_pendulum/pendubot.urdf (robot description, URDF)
Before this commit: robot double_pendulum, 6 links, 5 joints
Joints:
- joint joint1: limit lower=-10000 upper=10000 effort=0.1 velocity=25 -> lower=-10000 upper=10000 effort=0.1 velocity=20
- joint joint2: limit lower=-10000 upper=10000 effort=0.0 velocity=25 -> lower=-10000 upper=10000 effort=0.0 velocity=20

Commit message: Updated Pendubot solver benchmarks & added Go2 standing benchmarks

File: examples/assets/urdf/double_pendulum/pendubot.urdf (robot description, URDF)
Before this commit: robot double_pendulum, 6 links, 5 joints
Joints:
- joint joint1: limit lower=-10000 upper=10000 effort=0.1 velocity=20 -> lower=-10000 upper=10000 effort=0.1 velocity=10
- joint joint2: limit lower=-10000 upper=10000 effort=0.0 velocity=20 -> lower=-10000 upper=10000 effort=0.0 velocity=10
