Commit message: Updated Pendubot real MPC scripts & improved Python API for MPC

File: examples/assets/urdf/double_pendulum/acrobot.urdf (robot description, URDF)
Before this commit: robot double_pendulum, 6 links, 5 joints
Joints:
- joint joint1: limit lower=-10000 upper=10000 effort=0 velocity=40 -> lower=-10000 upper=10000 effort=0 velocity=20
- joint joint2: limit lower=-10000 upper=10000 effort=0.2 velocity=40 -> lower=-10000 upper=10000 effort=0.1 velocity=20

Commit message: Initial Acrobot real MPC script & minor SSQP output bug fix

File: examples/assets/urdf/double_pendulum/acrobot.urdf (robot description, URDF)
Before this commit: robot double_pendulum, 6 links, 5 joints
Joints:
- joint joint1: limit lower=-10000 upper=10000 effort=0 velocity=20 -> lower=-10000 upper=10000 effort=0 velocity=30
- joint joint2: limit lower=-10000 upper=10000 effort=0.1 velocity=20 -> lower=-10000 upper=10000 effort=0.1 velocity=30

Commit message: Further Acrobot tuning (1)

File: examples/assets/urdf/double_pendulum/acrobot.urdf (robot description, URDF)
Before this commit: robot double_pendulum, 6 links, 5 joints
Joints:
- joint joint2: limit lower=-10000 upper=10000 effort=0.1 velocity=30 -> lower=-10000 upper=10000 effort=0.14 velocity=30

Commit message: Fixed trajectory loading bugs

File: examples/assets/urdf/double_pendulum/acrobot.urdf (robot description, URDF)
Before this commit: robot double_pendulum, 6 links, 5 joints
Joints:
- joint joint2: limit lower=-10000 upper=10000 effort=0.14 velocity=30 -> lower=-10000 upper=10000 effort=0.1 velocity=30

File: examples/assets/urdf/double_pendulum/pendubot.urdf (robot description, URDF)
Before this commit: robot double_pendulum, 6 links, 5 joints
Joints:
- joint joint1: limit lower=-10000 upper=10000 effort=0.1 velocity=10 -> lower=-10000 upper=10000 effort=0.1 velocity=30
- joint joint2: limit lower=-10000 upper=10000 effort=0.0 velocity=10 -> lower=-10000 upper=10000 effort=0.0 velocity=30
