Commit message: Fixed HPIPM updating initial state bug (tolerance issue), added Go2 frog jumps example, added talos reduced model

File: examples/assets/urdf/go2/go2.urdf (robot description, URDF)
Before this commit: robot go2_description, 29 links, 28 joints
Joints:
- joint FL_foot_joint: origin xyz=0 0 -0.213 rpy=0 0 0 -> xyz=0 0 -0.235 rpy=0 0 0
- joint FR_foot_joint: origin xyz=0 0 -0.213 rpy=0 0 0 -> xyz=0 0 -0.235 rpy=0 0 0
- joint RL_foot_joint: origin xyz=0 0 -0.213 rpy=0 0 0 -> xyz=0 0 -0.235 rpy=0 0 0
- joint RR_foot_joint: origin xyz=0 0 -0.213 rpy=0 0 0 -> xyz=0 0 -0.235 rpy=0 0 0
