Commit message: Updated G1 URDF for force frames & added initial G1 examples

File: examples/assets/urdf/g1/g1_23dof.urdf (robot description, URDF)
Before this commit: robot g1_23dof, 33 links, 32 joints
Links:
- added link left_mm
- added link left_mp
- added link left_pm
- added link left_pp
- added link right_mm
- added link right_mp
- added link right_pm
- added link right_pp
Joints:
- added joint left_mm_fix_joint: type fixed, parent left_ankle_roll_link, child left_mm, origin xyz=-0.04 -0.03 -0.03 rpy=0 0 0
- added joint left_mp_fix_joint: type fixed, parent left_ankle_roll_link, child left_mp, origin xyz=-0.04 0.03 -0.03 rpy=0 0 0
- added joint left_pm_fix_joint: type fixed, parent left_ankle_roll_link, child left_pm, origin xyz=0.12 -0.03 -0.03 rpy=0 0 0
- added joint left_pp_fix_joint: type fixed, parent left_ankle_roll_link, child left_pp, origin xyz=0.12 0.03 -0.03 rpy=0 0 0
- added joint right_mm_fix_joint: type fixed, parent right_ankle_roll_link, child right_mm, origin xyz=-0.04 -0.03 -0.03 rpy=0 0 0
- added joint right_mp_fix_joint: type fixed, parent right_ankle_roll_link, child right_mp, origin xyz=-0.04 0.03 -0.03 rpy=0 0 0
- added joint right_pm_fix_joint: type fixed, parent right_ankle_roll_link, child right_pm, origin xyz=0.12 -0.03 -0.03 rpy=0 0 0
- added joint right_pp_fix_joint: type fixed, parent right_ankle_roll_link, child right_pp, origin xyz=0.12 0.03 -0.03 rpy=0 0 0
